File: Nexus-Kicad/Nexus.kicad_pcb (KiCad board)
At the start: 2 copper layers, 13 parts, among them J1 Conn_01x02_Socket

Commit message: add PCB
Parts:
- added BZ1: Buzzer, Buzzer_Beeper:Buzzer_15x7.5RM7.6, F.Cu at (151.9, 79.6)
- added C5: 10uF, Capacitor_SMD:C_0603_1608Metric, B.Cu at (98.7, 67.3)
- added D3: D_Schottky_Filled, Diode_THT:D_DO-201AE_P12.70mm_Horizontal, B.Cu at (103.1, 84.0)
- added D4: LED, LED_SMD:LED_0603_1608Metric, F.Cu at (95.7, 83.3)
- added D5: D_Schottky_Filled, Diode_THT:D_DO-201AD_P12.70mm_Horizontal, F.Cu at (115.5, 114.5)
- added D6: LED, LED_SMD:LED_0603_1608Metric, F.Cu at (96.3, 66.5)
- added D7: 1N4007, Diode_THT:D_DO-41_SOD81_P7.62mm_Horizontal, B.Cu at (143.3, 114.1)
- added D8: D, Diode_THT:D_DO-34_SOD68_P7.62mm_Horizontal, F.Cu at (136.1, 68.0)
- added J10: Conn_01x02_Socket, Connector_PinSocket_2.54mm:PinSocket_1x02_P2.54mm_Vertical, F.Cu at (145.2, 109.9)
- added J12: Conn_01x08_Socket, Connector_PinSocket_2.54mm:PinSocket_1x08_P2.54mm_Vertical, F.Cu at (161.8, 85.3)
- added J13: Conn_01x03_Socket, Connector_PinSocket_2.54mm:PinSocket_1x03_P2.54mm_Vertical, F.Cu at (137.5, 70.6)
- added J14: Conn_01x08_Socket, Connector_PinSocket_2.54mm:PinSocket_1x08_P2.54mm_Vertical, F.Cu at (159.2, 85.3)
- added J15: Conn_01x08_Socket, Connector_PinSocket_2.54mm:PinSocket_1x08_P2.54mm_Vertical, F.Cu at (156.7, 85.3)
- added J16: Conn_01x04_Socket, Connector_PinSocket_2.54mm:PinSocket_1x04_P2.54mm_Vertical, F.Cu at (125.7, 67.9)
- added J17: Conn_01x04_Socket, Connector_PinSocket_2.54mm:PinSocket_1x04_P2.54mm_Vertical, F.Cu at (125.7, 70.5)
- added J2: Conn_01x02_Pin, Connector_AMASS:AMASS_XT30U-F_1x02_P5.0mm_Vertical, F.Cu at (105.8, 100.9)
- added J3: Conn_01x02_Pin, Connector_AMASS:AMASS_XT30U-F_1x02_P5.0mm_Vertical, F.Cu at (99.4, 100.8)
- added J4: Conn_01x03_Socket, Connector_Molex:Molex_SPOX_5267-03A_1x03_P2.50mm_Vertical, F.Cu at (138.0, 112.9)
- added J5: Conn_01x03_Socket, Connector_Molex:Molex_SPOX_5267-03A_1x03_P2.50mm_Vertical, F.Cu at (126.7, 100.5)
- added J6: Conn_01x03_Socket, Connector_Molex:Molex_SPOX_5267-03A_1x03_P2.50mm_Vertical, F.Cu at (126.8, 106.7)
- added J7: Conn_01x03_Socket, Connector_Molex:Molex_SPOX_5267-03A_1x03_P2.50mm_Vertical, F.Cu at (126.8, 112.8)
- added MD1: OKL-T_6-W12N-C, OKLT6W12N:MURATA_OKL-T-6-W12N-C_0, F.Cu at (101.0, 75.3)
- added Q1: BSS138, Package_TO_SOT_SMD:SOT-23, F.Cu at (114.7, 95.9)
- added Q2: BSS138, Package_TO_SOT_SMD:SOT-23, B.Cu at (116.1, 95.9)
- added Q3: BSS138, Package_TO_SOT_SMD:SOT-23, B.Cu at (109.9, 95.9)
- added Q4: BSS138, Package_TO_SOT_SMD:SOT-23, F.Cu at (107.2, 95.7)
- added Q5: 2N7000, Package_TO_SOT_THT:TO-92_Inline, F.Cu at (150.2, 108.2)
- added R10: 2.2k, Resistor_SMD:R_0603_1608Metric, B.Cu at (117.7, 98.6)
- added R11: 2.2k, Resistor_SMD:R_0603_1608Metric, B.Cu at (111.7, 97.9)
- added R12: 2.2k, Resistor_SMD:R_0603_1608Metric, F.Cu at (110.8, 98.7)
- added R13: 1.2k, Resistor_SMD:R_0603_1608Metric, B.Cu at (109.0, 79.6)
- added R14: 1.2k, Resistor_SMD:R_0603_1608Metric, B.Cu at (97.1, 67.3)
- added R15: 1k, Resistor_SMD:R_0603_1608Metric, F.Cu at (96.3, 68.1)
- added R16: 1k, Resistor_SMD:R_0603_1608Metric, B.Cu at (152.2, 109.1)
- added R17: 10k, Resistor_SMD:R_0603_1608Metric, B.Cu at (148.2, 109.1)
- added R18: 1k, Resistor_SMD:R_0603_1608Metric, B.Cu at (104.3, 68.9)
- added R19: 1k, Resistor_SMD:R_0603_1608Metric, B.Cu at (104.3, 67.4)
- added R6: 2.2k, Resistor_SMD:R_0603_1608Metric, B.Cu at (113.3, 95.8)
- added R7: 2.2k, Resistor_SMD:R_0603_1608Metric, B.Cu at (107.1, 95.8)
- added R8: 2.2k, Resistor_SMD:R_0603_1608Metric, F.Cu at (110.1, 95.7)
- added R9: 2.2k, Resistor_SMD:R_0603_1608Metric, F.Cu at (113.2, 97.9)
- added U1: 74HC244D, 74HC244:SOIC20_TOS, F.Cu at (112.3, 88.2)
- added U2: TC7S14F_LF, tc7s14:SOT-25 SMV_TOS, B.Cu at (116.5, 88.7)
- added U3: RASPBERRY_PI_4B_4GB, RaspberryPi4B:MODULE_RASPBERRY_PI_4B_4GB, F.Cu at (136.9, 88.9)
- added U4: MCP3008, Package_DIP:DIP-16_W7.62mm_Socket, F.Cu at (153.3, 103.4)
- C1: value 22uF -> 470uF; footprint Capacitor_SMD:C_0603_1608Metric -> Capacitor_THT:CP_Radial_D10.0mm_P5.00mm
- C2: value 10uF -> 22uF
- C3: value 470uF -> 0.1uF; footprint Capacitor_THT:CP_Radial_D10.0mm_P5.00mm -> Capacitor_SMD:C_0603_1608Metric; moved to B.Cu
- C4: value 0.1uF -> 1000u; footprint Capacitor_SMD:C_0603_1608Metric -> Capacitor_THT:CP_Radial_D12.5mm_P5.00mm
- D1, D2: footprint LED_SMD:LED_0603_1608Metric_Pad1.05x0.95mm_HandSolder -> LED_SMD:LED_0603_1608Metric
- J1: footprint Connector_AMASS:AMASS_XT60-F_1x02_P7.20mm_Vertical -> Connector_AMASS:AMASS_XT30U-F_1x02_P5.0mm_Vertical
- R1: value 20k -> 2k
- R2, R3: value 1.2k -> 2k
- R4: value 2k -> 20k; moved to B.Cu
- R5: value 1k -> 2.2k
- RV1: moved to B.Cu
- moved C4 53.9 mm to (133.9, 104.0)
- moved D1 44.5 mm to (95.7, 101.7), turned to -90 degrees
- moved R1 42.2 mm to (95.7, 104.9), turned to 90 degrees
- moved D2 39.7 mm to (109.7, 107.0), turned to 90 degrees
- moved R2 39.0 mm to (109.7, 103.9), turned to -90 degrees
- moved C1 32.6 mm to (100.1, 88.1), turned to -90 degrees
- moved J1 32.5 mm to (109.4, 112.9), turned to 180 degrees
- moved R5 27.5 mm to (117.5, 95.8), turned to 90 degrees
- moved C3 25.0 mm to (96.4, 82.5), turned to 180 degrees
- moved C2 24.7 mm to (98.0, 82.5), turned to 180 degrees
- moved RV1 18.1 mm to (109.0, 72.5), turned to -90 degrees
- moved R3 16.2 mm to (98.0, 83.9), turned to 180 degrees
- moved R4 14.3 mm to (96.5, 83.9), turned to 180 degrees
Connections:
- C1 pad 2: GNDD -> GNDA
- C2 pad 1: +5V -> Net-(D3-K)
- C2 pad 2: GNDD -> GNDA
- C3 pad 2: GNDD -> GNDA
- C4 pad 1: Net-(D3-K) -> V-Servo
- C4 pad 2: GNDD -> GNDA
- D1 pad 1: GNDD -> GNDA
- D2 pad 1: GNDD -> GNDA
- J1 pad 1: unconnected-(J1-Pin_1-Pad1) -> GNDA
- J1 pad 2: Vcc -> batte
- R1 pad 1: Net-(D3-K) -> batte
- R1 pad 2: GNDD -> Net-(D1-A)
- R2 pad 1: +5V -> +12V
- R2 pad 2: GNDD -> Net-(D2-A)
- R3 pad 1: Net-(R3-Pad1) -> Net-(D3-K)
- R3 pad 2: GNDD -> Net-(D4-A)
- R4 pad 2: Net-(D1-A) -> GNDA
- R5 pad 1: +5V -> 3.3V
- R5 pad 2: Net-(D2-A) -> Servo1_3.3V
- RV1 pad 2: Net-(R3-Pad1) -> Net-(R13-Pad1)
Routing:
- net 3.3V: track 0.00 -> 150.3 mm, vias 0 -> 4
- net RX4: track 0.00 -> 48.2 mm, vias 0 -> 1
- net RX3: track 0.00 -> 47.6 mm, vias 0 -> 1
- net Fan_PWM: track 0.00 -> 45.1 mm, vias 0 -> 1
- net Dout: track 0.00 -> 43.7 mm, vias 0 -> 2
- net Cs: track 0.00 -> 42.2 mm
- net Clock: track 0.00 -> 40.3 mm
- net TX2: track 0.00 -> 39.6 mm
- net RX2: track 0.00 -> 37.3 mm, vias 0 -> 1
- net +5V: track 0.00 -> 35.0 mm, vias 0 -> 51
- net DIn: track 0.00 -> 34.9 mm, vias 0 -> 2
- net Servo1_5V: track 0.00 -> 33.9 mm
- net Enable: track 0.00 -> 33.3 mm, vias 0 -> 3
- net Servo4_5V: track 0.00 -> 29.1 mm
- net Net-(D3-K): track 0.00 -> 26.9 mm, vias 0 -> 1
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- added copper zone on In2.Cu, net +5V
- added copper zone on In4.Cu, net +5V
- added copper zone on B.Cu, net GNDA
- added copper zone on F.Cu, net GNDA
- added copper zone on In1.Cu, net GNDA
- added copper zone on In3.Cu, net GNDA
- added copper zone on In2.Cu, net V-Servo
- added copper zone on In4.Cu, net V-Servo
Other:
- board outline added: 69.5 x 56 mm
- copper layers 2 -> 6
- board text added: "B.T.F-Nexus"
- board text added: "ver 1.0"

Commit message: JLCPCB
Parts:
- D7: moved to F.Cu
- moved D6 3.35 mm to (99.3, 68.1)
- moved C5 2.54 mm to (96.3, 68.1), turned to 180 degrees
- moved R14 2.44 mm to (99.4, 68.1), turned to 0 degrees
- moved MD1 0.38 mm to (101.3, 75.4)
- moved D5 0.20 mm to (115.6, 114.3)
- moved J16 0.07 mm to (125.7, 68.0)
- moved J17 0.07 mm to (125.7, 70.5)
- moved R15 0.06 mm to (96.2, 68.1), turned to 0 degrees
Routing:
- net +5V: track 35.0 -> 38.9 mm, vias 51 -> 43
- net 3.3V: track 150.3 -> 149.2 mm
- net Enable: track 33.3 -> 32.6 mm
- net V-Servo: vias 18 -> 16
- net GNDA: vias 73 -> 63
Other:
- board size 69.5 x 56 mm -> 69.5 x 56.1 mm

Commit message: ver2
Parts:
- removed the C4 at (133.9, 104.0)
- removed the J4 at (138.0, 112.9)
- removed J5: Conn_01x03_Socket, Connector_Molex:Molex_SPOX_5267-03A_1x03_P2.50mm_Vertical
- removed the J6 at (126.8, 106.7)
- removed the J7 at (126.8, 112.8)
- added C5: 470u, Capacitor_THT:CP_Radial_D10.0mm_P5.00mm, F.Cu at (146.6, 107.8)
- added J12: Conn_01x03_Socket, Connector_PinHeader_2.54mm:PinHeader_1x03_P2.54mm_Vertical, F.Cu at (120.0, 104.7)
- added J13: Conn_01x03_Socket, Connector_PinHeader_2.54mm:PinHeader_1x03_P2.54mm_Vertical, F.Cu at (122.5, 104.7)
- added J14: Conn_01x03_Socket, Connector_PinHeader_2.54mm:PinHeader_1x03_P2.54mm_Vertical, F.Cu at (125.1, 104.7)
- added J15: Conn_01x03_Socket, Connector_PinHeader_2.54mm:PinHeader_1x03_P2.54mm_Vertical, F.Cu at (127.6, 104.7)
- added J16: Conn_01x03_Socket, Connector_PinHeader_2.54mm:PinHeader_1x03_P2.54mm_Vertical, F.Cu at (132.0, 104.7)
- added J17: Conn_01x03_Socket, Connector_PinHeader_2.54mm:PinHeader_1x03_P2.54mm_Vertical, F.Cu at (134.5, 104.7)
- added J18: Conn_01x03_Socket, Connector_PinHeader_2.54mm:PinHeader_1x03_P2.54mm_Vertical, F.Cu at (137.1, 104.7)
- added J19: Conn_01x03_Socket, Connector_PinHeader_2.54mm:PinHeader_1x03_P2.54mm_Vertical, F.Cu at (139.6, 104.7)
- added J20: Conn_01x03_Socket, Connector_PinHeader_2.54mm:PinHeader_1x03_P2.54mm_Vertical, F.Cu at (119.9, 109.6)
- added J21: Conn_01x03_Socket, Connector_PinHeader_2.54mm:PinHeader_1x03_P2.54mm_Vertical, F.Cu at (122.5, 109.6)
- added J22: Conn_01x03_Socket, Connector_PinHeader_2.54mm:PinHeader_1x03_P2.54mm_Vertical, F.Cu at (125.0, 109.6)
- added J23: Conn_01x03_Socket, Connector_PinHeader_2.54mm:PinHeader_1x03_P2.54mm_Vertical, F.Cu at (127.6, 109.6)
- added J24: Conn_01x03_Socket, Connector_PinHeader_2.54mm:PinHeader_1x03_P2.54mm_Vertical, F.Cu at (132.0, 109.6)
- added J25: Conn_01x03_Socket, Connector_PinHeader_2.54mm:PinHeader_1x03_P2.54mm_Vertical, F.Cu at (134.5, 109.6)
- added J26: Conn_01x03_Socket, Connector_PinHeader_2.54mm:PinHeader_1x03_P2.54mm_Vertical, F.Cu at (137.1, 109.6)
- added J27: Conn_01x03_Socket, Connector_PinHeader_2.54mm:PinHeader_1x03_P2.54mm_Vertical, F.Cu at (139.6, 109.6)
- moved R18 17.6 mm to (121.4, 73.5), turned to 180 degrees
- moved R19 17.1 mm to (119.6, 75.1), turned to 180 degrees
- moved R17 13.3 mm to (161.4, 109.9)
- moved J2 12.5 mm to (108.7, 113.1), turned to 180 degrees
- moved J1 12.4 mm to (105.8, 101.0), turned to -90 degrees
- moved D6 10.9 mm to (151.6, 107.1), turned to -90 degrees
- moved J4 9.74 mm to (154.6, 107.5), turned to 0 degrees
- moved Q5 9.53 mm to (159.7, 109.1)
- moved R16 4.86 mm to (157.0, 109.5)
- moved J7 3.91 mm to (141.4, 71.2), turned to -90 degrees
- moved R2 3.13 mm to (109.7, 107.0), turned to 90 degrees
- moved D2 3.08 mm to (109.7, 103.9), turned to -90 degrees
- moved D7 1.13 mm to (135.0, 68.4)
- moved J10 0.77 mm to (125.5, 68.7)
- moved J11 0.77 mm to (125.5, 71.2)
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- renumbered C5 to C4, D6 to D5, D7 to D6, D8 to D7, D5 to D8, J16 to J10, J17 to J11, J10 to J4, J12 to J6, J13 to J7, J14 to J8, J15 to J9, Q4 to Q3, Q3 to Q4, R12 to R11, R11 to R12, R8 to R7, R7 to R8
Connections:
- net RX1 renamed RXD0
- net RX3 renamed RXD3
- net TX1 renamed TXD0
- net TX3 renamed TXD3
- U1 pad 2: TX4 -> TXD5
- U1 pad 3: RX4 -> RXD5
- U1 pad 4: TX2 -> TXD4
- U1 pad 5: RX2 -> RXD4
- U3 pad 11: Enable -> Cs
- U3 pad 12: unconnected-(U3-GPIO18/GPIO_GEN1-Pad12) -> FLED_Sig
- U3 pad 13: unconnected-(U3-GPIO27/GPIO_GEN2-Pad13) -> Enable
- U3 pad 18: TX4 -> unconnected-(U3-GPIO24/GPIO_GEN5-Pad18)
- U3 pad 19: DIn -> unconnected-(U3-GPIO10/SPI_MOSI-Pad19)
- U3 pad 21: Dout -> RXD4
- U3 pad 24: Cs -> TXD4
- U3 pad 26: Clock -> unconnected-(U3-GPIO7/~{SPI_CE1}-Pad26)
- U3 pad 27: TX2 -> unconnected-(U3-ID_SD-Pad27)
- U3 pad 28: RX2 -> unconnected-(U3-ID_SC-Pad28)
- U3 pad 32: Sig_Buzzer -> TXD5
- U3 pad 33: FLED_Sig -> RXD5
- U3 pad 35: Fan_PWM -> Dout
- U3 pad 36: unconnected-(U3-GPIO16-Pad36) -> Fan_PWM
- U3 pad 37: unconnected-(U3-GPIO26-Pad37) -> Sig_Buzzer
- U3 pad 38: unconnected-(U3-GPIO20-Pad38) -> DIn
- U3 pad 40: RX4 -> Clock
Routing:
- net V-Servo: track 0.00 -> 110.6 mm, vias 16 -> 0
- net RX4: track 48.2 -> 0.00 mm, vias 1 -> 0
- net TX2: track 39.6 -> 0.00 mm
- net RX2: track 37.3 -> 0.00 mm, vias 1 -> 0
- net TXD5: track 0.00 -> 37.1 mm
- net TXD4: track 0.00 -> 36.0 mm
- net RXD5: track 0.00 -> 35.1 mm, vias 0 -> 1
- net RXD4: track 0.00 -> 30.4 mm, vias 0 -> 1
- net TX4: track 26.1 -> 0.00 mm
- net +5V: track 38.9 -> 19.5 mm, vias 43 -> 2
- net FLED_Sig: track 5.98 -> 24.8 mm
- net Servo2_5V: track 10.1 -> 28.7 mm
- net Fan_PWM: track 45.1 -> 63.4 mm, vias 1 -> 0
- net Sig_Buzzer: track 22.6 -> 7.25 mm
- net Dout: track 43.7 -> 28.3 mm, vias 2 -> 0
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Other:
- outline, holes or cut-outs redrawn
- board text added: "Nexus"
- board text removed: "B.T.F-Nexus"
- board text removed: "ver 1.0"
